File: Phase_B/Uno_Shield_ThermoPro/Uno_Shield_ThermoPro.kicad_pcb (KiCad board)
At the start: 2 copper layers, 68.6 x 53.3 mm, 20 parts, among them J1 Power, J2 Digital/PWM, J3 Analog, J4 Digital/PWM, J5 CONN_GYRO, J6 CONN_DISPLAY, J7 CONN_TEMP, SW1 SW_SPST, SW2 SW_SPST, SW3 SW_SPST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

Commit message: 02-02-2025 18:40 Updating Finalized Files
Routing:
- net /temp_sensor: track 13.7 -> 11.8 mm
- net /button_cal: track 70.9 -> 71.6 mm
Other:
- board text added: "Cal Button"
- board text added: "Light Button"
- board text added: "Lock Button"
- board text added: "On/Off"
- board text added: "Units Button"
Changed lines of the file:
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@@
 		(tags "connector JST XH vertical")
 		(property "Reference" "J7"
-			(at 2.5 -3.55 0)
+			(at 2.27 4.82 0)
 			(layer "F.SilkS")
 			(effects
@@
 		)
 	)
+	(gr_text "Light Button"
+		(at 145 93.5 0)
+		(layer "F.SilkS")
+		(effects
+			(font
+				(size 1 1)
+				(thickness 0.15)
+			)
+			(justify left bottom)
+		)
+	)
+	(gr_text "Units Button"
+		(at 130.5 78.5 0)
+		(layer "F.SilkS")
+		(effects
+			(font
+				(size 1 1)
+				(thickness 0.15)
+			)
+			(justify left bottom)
+		)
+	)
+	(gr_text "Cal Button"
+		(at 130.5 93.5 0)
+		(layer "F.SilkS")
+		(effects
+			(font
+				(size 1 1)
+				(thickness 0.15)
+			)
+			(justify left bottom)
+		)
+	)
+	(gr_text "On/Off"
+		(at 146 77.5 0)
+		(layer "F.SilkS")
+		(effects
+			(font
+				(size 1 1)
+				(thickness 0.15)
+			)
+			(justify left bottom)
+		)
+	)
+	(gr_text "Lock Button"
+		(at 157.5 81.5 0)
+		(layer "F.SilkS")
+		(effects
+			(font
+				(size 1 1)
+				(thickness 0.15)
+			)
+			(justify left bottom)
+		)
+	)
 	(segment
 		(start 128.846 62.224)
@@
 	)
 	(segment
-		(start 142.67 90.17)
-		(end 142.67 82.056576)
+		(start 158.03 78.36)
+		(end 157.39 79)
+		(width 0.508)
+		(layer "F.Cu")
+		(net 3)
+	)
+	(segment
+		(start 145.726576 79)
+		(end 143.216 81.510576)
 		(width 0.508)
 		(layer "F.Cu")
@@
 	)
 	(segment
+		(start 143 90.17)
+		(end 146.25 90.17)
+		(width 0.508)
+		(layer "F.Cu")
+		(net 3)
+	)
+	(segment
 		(start 129.566 77.234)
 		(end 129.566 87.266)
@@
 	)
 	(segment
+		(start 142.67 90.17)
+		(end 143 90.17)
+		(width 0.508)
+		(layer "F.Cu")
+		(net 3)
+	)
+	(segment
 		(start 128.95 75.14)
 		(end 131.66 75.14)
@@
 	)
 	(segment
+		(start 157.39 79)
+		(end 145.726576 79)
+		(width 0.508)
+		(layer "F.Cu")
+		(net 3)
+	)
+	(segment
 		(start 146.26 90.18)
 		(end 152.76 90.18)
@@
 	)
 	(segment
-		(start 146.25 90.17)
-		(end 146.26 90.18)
+		(start 143.216 81.510576)
+		(end 143.216 89.954)
 		(width 0.508)
 		(layer "F.Cu")
@@
 	)
 	(segment
-		(start 146.366576 78.36)
-		(end 158.03 78.36)
+		(start 146.25 90.17)
+		(end 146.26 90.18)
 		(width 0.508)
 		(layer "F.Cu")
@@
 	)
 	(segment
-		(start 142.67 82.056576)
-		(end 146.366576 78.36)
-		(width 0.508)
-		(layer "F.Cu")
-		(net 3)
-	)
-	(segment
-		(start 142.67 90.17)
-		(end 146.25 90.17)
+		(start 143.216 89.954)
+		(end 143 90.17)
 		(width 0.508)
 		(layer "F.Cu")
@@
 	)
 	(segment
-		(start 139.436267 75.92)
-		(end 154.05 75.92)
+		(start 154.728 75.772)
+		(end 152.208 78.292)
+		(width 0.508)
+		(layer "F.Cu")
+		(net 20)
+	)
+	(segment
+		(start 132.5 80)
+		(end 132.5 80.28)
+		(width 0.508)
+		(layer "F.Cu")
+		(net 20)
+	)
+	(segment
+		(start 145.433312 78.292)
+		(end 143.725312 80)
+		(width 0.508)
+		(layer "F.Cu")
+		(net 20)
+	)
+	(segment
+		(start 154.728 75)
+		(end 154.728 67.062)
+		(width 0.508)
+		(layer "F.Cu")
+		(net 20)
+	)
+	(segment
+		(start 154.728 75)
+		(end 154.728 75.772)
 		(width 0.508)
 		(layer "F.Cu")
@@
 	)
 	(segment
+		(start 132.5 80.28)
+		(end 130.82 81.96)
+		(width 0.508)
+		(layer "F.Cu")
+		(net 20)
+	)
+	(segment
 		(start 155.274 65.454)
 		(end 155.18 65.36)
@@
 	)
 	(segment
-		(start 154.05 75.92)
-		(end 154.728 75.242)
+		(start 152.208 78.292)
+		(end 145.433312 78.292)
 		(width 0.508)
 		(layer "F.Cu")
@@
 	)
 	(segment
-		(start 133.396267 81.96)
-		(end 139.436267 75.92)
-		(width 0.508)
-		(layer "F.Cu")
-		(net 20)
-	)
-	(segment
-		(start 130.82 81.96)
-		(end 133.396267 81.96)
+		(start 143.725312 80)
+		(end 132.5 80)
 		(width 0.508)
 		(layer "F.Cu")
@@
 	)
 	(segment
-		(start 160.47 60.07)
-		(end 160.47 54.397472)
+		(start 154.728 75.242)
+		(end 154.728 75)
 		(width 0.508)
 		(layer "F.Cu")
@@
 	)
 	(segment
-		(start 154.728 75.242)
-		(end 154.728 67.062)
+		(start 160.47 60.07)
+		(end 160.47 54.397472)
 		(width 0.508)
 		(layer "F.Cu")
@@
 	)
 	(segment
-		(start 160.44 92.3)
-		(end 152.65 92.3)
+		(start 153.26 95)
+		(end 156.5 95)
+		(width 0.508)
+		(layer "F.Cu")
+		(net 23)
+	)
+	(segment
+		(start 150.8 97.46)
+		(end 153.26 95)
 		(width 0.508)
 		(layer "F.Cu")
@@
 	)
 	(segment
-		(start 150.8 94.15)
-		(end 150.8 97.46)
+		(start 156.5 95)
+		(end 159.2 92.3)
 		(width 0.508)
 		(layer "F.Cu")
@@
 	)
 	(segment
-		(start 152.65 92.3)
-		(end 150.8 94.15)
+		(start 159.2 92.3)
+		(end 160.44 92.3)
 		(width 0.508)
 		(layer "F.Cu")
