File: Phase_B/Uno_Shield_ThermoPro/Uno_Shield_ThermoPro.kicad_pcb (KiCad board)
At the start: 2 copper layers, 68.6 x 53.3 mm, 20 parts, among them J1 Power, J2 Digital/PWM, J3 Analog, J4 Digital/PWM, J5 CONN_GYRO, J6 CONN_DISPLAY, J7 CONN_TEMP, SW1 SW_SPST, SW2 SW_SPST, SW3 SW_SPST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

Commit message: 02-03-2025 18:56 Updating files for Phase B.
Parts:
- added G***: LOGO, LOGO, F.Cu at (105.5, 95.0)
- moved D1 2.96 mm to (153.5, 59.5), turned to 180 degrees
- moved J7 0.32 mm to (139.1, 56.7)
Routing:
- net Net-(D1-A): track 26.6 -> 19.9 mm
- net /button_units: track 52.3 -> 48.7 mm
- net /button_onoff: track 37.5 -> 34.6 mm
- net /button_light: track 69.1 -> 66.4 mm
- net /button_cal: track 71.4 -> 69.2 mm
- net +5V: track 167.5 -> 165.8 mm
- net /button_lock: track 36.8 -> 35.4 mm
- net /temp_sensor: track 11.8 -> 12.5 mm
Other:
- board text added: "+5V"
- board text added: "2"
- board text added: "3"
- board text added: "4"
- board text added: "5"
- board text added: "6"
- board text added: "8"
- board text added: "9"
- board text added: "Analog Sensor"
- board text added: "Temp Sensor"
- board text added: "ThermoProbe Version 1 02-03-2025 Braidyn Sheffield"
