File: Phase_B/Uno_Shield_ThermoPro/Uno_Shield_ThermoPro.kicad_sch (KiCad schematic)
At the start: 20 parts, among them J1 Power, J2 Digital/PWM, J3 Analog, J4 Digital/PWM, J5 CONN_GYRO, J6 CONN_DISPLAY, J7 CONN_TEMP, SW1 SW_SPST, SW2 SW_SPST, SW3 SW_SPST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

Commit message: 02-03-2025 18:56 Updating files for Phase B.
Changed lines of the file:
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@@
 	)
 	(label "temp_sensor"
-		(at 30.48 59.69 180)
+		(at 29.21 59.69 180)
 		(effects
 			(font
